File: KiCad/Main/Moteurs et alimentation.kicad_sch (KiCad schematic)
At the start: 11 parts, among them J10 Conn_01x02_Pin, J11 Conn_01x10_Pin, J9 Conn_01x02_Pin, SW1 SW_DPST

Commit message: ok
Parts:
- J10, J9: footprint (none) -> Connector_JST:JST_EH_B2B-EH-A_1x02_P2.50mm_Vertical
- J11: footprint (none) -> Connector_JST:JST_EH_B10B-EH-A_1x10_P2.50mm_Vertical
Changed lines of the file:
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@@
 			)
 		)
-		(property "Footprint" ""
+		(property "Footprint" "Connector_JST:JST_EH_B10B-EH-A_1x10_P2.50mm_Vertical"
 			(at 262.89 115.57 0)
 			(effects
@@
 			)
 		)
-		(property "Footprint" ""
+		(property "Footprint" "Connector_JST:JST_EH_B2B-EH-A_1x02_P2.50mm_Vertical"
 			(at 262.89 74.93 0)
 			(effects
@@
 			)
 		)
-		(property "Footprint" ""
+		(property "Footprint" "Connector_JST:JST_EH_B2B-EH-A_1x02_P2.50mm_Vertical"
 			(at 262.89 67.31 0)
 			(effects
