File: KiCad/Main/main.kicad_pcb (KiCad board)
At the start: 2 copper layers, 18 parts, among them J1 Vers GPS, J10 Conn_01x02_Pin, J11 Conn_01x10_Pin, J2 Vers Moteurs, J3 Vers Display, J4 Vers GPS, J5 Conn_01x02_Pin, J6 Conn_01x02_Pin, J7 RJ45, J8 RJ45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

Commit message: ok
Parts:
- moved J2 97.8 mm to (48.5, 37.5)
Connections:
- net /Moteurs et alimentation/ALT/DIR renamed /Moteurs/ALT/DIR
- net /Moteurs et alimentation/ALT/STEP renamed /Moteurs/ALT/STEP
- net /Moteurs et alimentation/AZ/DIR renamed /Moteurs/AZ/DIR
- net /Moteurs et alimentation/AZ/STEP renamed /Moteurs/AZ/STEP
- net /Moteurs et alimentation/EN renamed /Moteurs/EN
- net /Moteurs et alimentation/M0 renamed /Moteurs/M0
- net /Moteurs et alimentation/M1 renamed /Moteurs/M1
- net /Moteurs et alimentation/M2 renamed /Moteurs/M2
- net /Moteurs et alimentation/RST/SLP renamed /Moteurs/RST/SLP
- A1 pad 1: /Moteurs et alimentation/GND -> /Moteurs/GND
- A2 pad 1: /Moteurs et alimentation/GND -> /Moteurs/GND
- J11 pad 1: /Moteurs et alimentation/PontDiviseur -> /Moteurs/GND
- J2 pad 1: /PontDiviseur -> /GND
- U5 pad 41: /PontDiviseur -> Net-(U5-GPIO1/ADC1_CH0)
Changed lines of the file:
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@@
 	(net 1 "unconnected-(A1-~{FLT}-Pad2)")
 	(net 2 "unconnected-(A1-A1-Pad4)")
-	(net 3 "/Moteurs et alimentation/RST{slash}SLP")
+	(net 3 "/Moteurs/RST{slash}SLP")
 	(net 4 "Net-(A1-VMOT)")
-	(net 5 "/Moteurs et alimentation/M1")
-	(net 6 "/Moteurs et alimentation/M0")
+	(net 5 "/Moteurs/M1")
+	(net 6 "/Moteurs/M0")
 	(net 7 "unconnected-(A1-B1-Pad5)")
-	(net 8 "/Moteurs et alimentation/ALT{slash}DIR")
+	(net 8 "/Moteurs/ALT{slash}DIR")
 	(net 9 "unconnected-(A1-A2-Pad3)")
 	(net 10 "unconnected-(A1-B2-Pad6)")
-	(net 11 "/Moteurs et alimentation/M2")
-	(net 12 "/Moteurs et alimentation/ALT{slash}STEP")
+	(net 11 "/Moteurs/M2")
+	(net 12 "/Moteurs/ALT{slash}STEP")
 	(net 13 "/Moteurs et alimentation/GND")
-	(net 14 "Net-(LM1-IN-)")
-	(net 15 "/Moteurs et alimentation/EN")
+	(net 14 "/Moteurs/GND")
+	(net 15 "Net-(J5-Pin_5)")
 	(net 16 "unconnected-(A2-B2-Pad6)")
 	(net 17 "unconnected-(A2-B1-Pad5)")
 	(net 18 "unconnected-(A2-A1-Pad4)")
 	(net 19 "unconnected-(A2-A2-Pad3)")
-	(net 20 "/Moteurs et alimentation/AZ{slash}DIR")
-	(net 21 "/Moteurs et alimentation/AZ{slash}STEP")
+	(net 20 "/Moteurs/EN")
+	(net 21 "/Moteurs/AZ{slash}DIR")
 	(net 22 "unconnected-(A2-~{FLT}-Pad2)")
 	(net 23 "Net-(U3-GND)")
 	(net 24 "Net-(U3-VCC)")
 	(net 25 "/ALT{slash}STEP")
-	(net 26 "/PontDiviseur")
+	(net 26 "/Moteurs/AZ{slash}STEP")
 	(net 27 "/M1")
 	(net 28 "/RST{slash}SLP")
@@
 	(net 49 "/SDA")
 	(net 50 "/Moteurs et alimentation/5V")
-	(net 51 "/Moteurs et alimentation/PontDiviseur")
+	(net 51 "Net-(U5-GPIO1{slash}ADC1_CH0)")
 	(net 52 "/RST")
 	(net 53 "/TXD")
@@
 		)
 		(property ki_fp_filters "CP_*")
-		(sheetname "/Moteurs et alimentation/")
+		(sheetname "/Moteurs/")
 		(sheetfile "Moteurs et alimentation.kicad_sch")
 		(attr through_hole)
@@
 			(layers "*.Cu" "*.Mask")
 			(remove_unused_layers no)
-			(net 14 "Net-(LM1-IN-)")
+			(net 15 "Net-(J5-Pin_5)")
 			(pintype "passive")
 		)
@@
 	(footprint "Connector_JST:JST_EH_B10B-EH-A_1x10_P2.50mm_Vertical"
 		(layer "F.Cu")
-		(at 146 44.5 -90)
+		(at 48.5 37.5 -90)
 		(descr "JST EH series connector, B10B-EH-A (http://www.jst-mfg.com/product/pdf/eng/eEH.pdf), generated with kicad-footprint-generator")
 		(tags "connector JST EH vertical")
@@
 			(remove_unused_layers no)
 			(roundrect_rratio 0.147059)
-			(net 26 "/PontDiviseur")
+			(net 36 "/GND")
 			(pinfunction "Pin_1")
 			(pintype "passive")
@@
 		)
 		(property ki_fp_filters "Connector*:*_1x??_*")
-		(sheetname "/Moteurs et alimentation/")
+		(sheetname "/Moteurs/")
 		(sheetfile "Moteurs et alimentation.kicad_sch")
 		(attr through_hole)
@@
 			(remove_unused_layers no)
 			(roundrect_rratio 0.147059)
-			(net 51 "/Moteurs et alimentation/PontDiviseur")
+			(net 14 "/Moteurs/GND")
 			(pinfunction "Pin_1")
 			(pintype "passive")
@@
 			(layers "*.Cu" "*.Mask")
 			(remove_unused_layers no)
-			(net 6 "/Moteurs et alimentation/M0")
+			(net 6 "/Moteurs/M0")
 			(pinfunction "Pin_2")
 			(pintype "passive")
@@
 			(layers "*.Cu" "*.Mask")
 			(remove_unused_layers no)
-			(net 5 "/Moteurs et alimentation/M1")
+			(net 5 "/Moteurs/M1")
 			(pinfunction "Pin_3")
 			(pintype "passive")
@@
 			(layers "*.Cu" "*.Mask")
 			(remove_unused_layers no)
-			(net 11 "/Moteurs et alimentation/M2")
+			(net 11 "/Moteurs/M2")
 			(pinfunction "Pin_4")
 			(pintype "passive")
@@
 			(layers "*.Cu" "*.Mask")
 			(remove_unused_layers no)
-			(net 3 "/Moteurs et alimentation/RST{slash}SLP")
+			(net 3 "/Moteurs/RST{slash}SLP")
 			(pinfunction "Pin_5")
 			(pintype "passive")
@@
 			(layers "*.Cu" "*.Mask")
 			(remove_unused_layers no)
-			(net 15 "/Moteurs et alimentation/EN")
+			(net 20 "/Moteurs/EN")
 			(pinfunction "Pin_6")
 			(pintype "passive")
@@
 			(layers "*.Cu" "*.Mask")
 			(remove_unused_layers no)
-			(net 21 "/Moteurs et alimentation/AZ{slash}STEP")
+			(net 26 "/Moteurs/AZ{slash}STEP")
 			(pinfunction "Pin_7")
 			(pintype "passive")
@@
 			(layers "*.Cu" "*.Mask")
 			(remove_unused_layers no)
-			(net 20 "/Moteurs et alimentation/AZ{slash}DIR")
+			(net 21 "/Moteurs/AZ{slash}DIR")
 			(pinfunction "Pin_8")
 			(pintype "passive")
@@
 			(layers "*.Cu" "*.Mask")
 			(remove_unused_layers no)
-			(net 12 "/Moteurs et alimentation/ALT{slash}STEP")
+			(net 12 "/Moteurs/ALT{slash}STEP")
 			(pinfunction "Pin_9")
 			(pintype "passive")
@@
 			(layers "*.Cu" "*.Mask")
 			(remove_unused_layers no)
-			(net 8 "/Moteurs et alimentation/ALT{slash}DIR")
+			(net 8 "/Moteurs/ALT{slash}DIR")
 			(pinfunction "Pin_10")
 			(pintype "passive")
@@
 		)
 		(property ki_fp_filters "CP_*")
-		(sheetname "/Moteurs et alimentation/")
+		(sheetname "/Moteurs/")
 		(sheetfile "Moteurs et alimentation.kicad_sch")
 		(attr through_hole)
@@
 			(layers "*.Cu" "*.Mask")
 			(remove_unused_layers no)
-			(net 14 "Net-(LM1-IN-)")
+			(net 15 "Net-(J5-Pin_5)")
 			(pintype "passive")
 		)
@@
 		)
 		(property ki_fp_filters "Pololu*Breakout*15.2x20.3mm*")
-		(sheetname "/Moteurs et alimentation/")
+		(sheetname "/Moteurs/")
 		(sheetfile "Moteurs et alimentation.kicad_sch")
 		(attr through_hole)
@@
 			(layers "*.Cu" "*.Mask")
 			(remove_unused_layers no)
-			(net 13 "/Moteurs et alimentation/GND")
+			(net 14 "/Moteurs/GND")
 			(pinfunction "GND")
 			(pintype "power_in")
@@
 			(layers "*.Cu" "*.Mask")
 			(remove_unused_layers no)
-			(net 14 "Net-(LM1-IN-)")
+			(net 15 "Net-(J5-Pin_5)")
 			(pinfunction "GND")
 			(pintype "power_in")
@@
 			(layers "*.Cu" "*.Mask")
 			(remove_unused_layers no)
-			(net 15 "/Moteurs et alimentation/EN")
+			(net 20 "/Moteurs/EN")
 			(pinfunction "~{EN}")
 			(pintype "input")
@@
 			(layers "*.Cu" "*.Mask")
 			(remove_unused_layers no)
-			(net 6 "/Moteurs et alimentation/M0")
+			(net 6 "/Moteurs/M0")
 			(pinfunction "M0")
 			(pintype "input")
@@
 			(layers "*.Cu" "*.Mask")
 			(remove_unused_layers no)
-			(net 5 "/Moteurs et alimentation/M1")
+			(net 5 "/Moteurs/M1")
 			(pinfunction "M1")
 			(pintype "input")
@@
 			(layers "*.Cu" "*.Mask")
 			(remove_unused_layers no)
-			(net 11 "/Moteurs et alimentation/M2")
+			(net 11 "/Moteurs/M2")
 			(pinfunction "M2")
 			(pintype "input")
@@
 			(layers "*.Cu" "*.Mask")
 			(remove_unused_layers no)
-			(net 3 "/Moteurs et alimentation/RST{slash}SLP")
+			(net 3 "/Moteurs/RST{slash}SLP")
 			(pinfunction "~{RST}")
 			(pintype "input")
@@
 			(layers "*.Cu" "*.Mask")
 			(remove_unused_layers no)
-			(net 3 "/Moteurs et alimentation/RST{slash}SLP")
+			(net 3 "/Moteurs/RST{slash}SLP")
 			(pinfunction "~{SLP}")
 			(pintype "input")
@@
 			(layers "*.Cu" "*.Mask")
 			(remove_unused_layers no)
-			(net 21 "/Moteurs et alimentation/AZ{slash}STEP")
+			(net 26 "/Moteurs/AZ{slash}STEP")
 			(pinfunction "STEP")
 			(pintype "input")
@@
 			(layers "*.Cu" "*.Mask")
 			(remove_unused_layers no)
-			(net 20 "/Moteurs et alimentation/AZ{slash}DIR")
+			(net 21 "/Moteurs/AZ{slash}DIR")
 			(pinfunction "DIR")
 			(pintype "input")
@@
 			(layers "*.Cu" "*.Mask")
 			(remove_unused_layers no)
-			(net 26 "/PontDiviseur")
+			(net 51 "Net-(U5-GPIO1{slash}ADC1_CH0)")
 			(pinfunction "GPIO1/ADC1_CH0")
 			(pintype "bidirectional")
@@
 		)
 		(property ki_fp_filters "Pololu*Breakout*15.2x20.3mm*")
-		(sheetname "/Moteurs et alimentation/")
+		(sheetname "/Moteurs/")
 		(sheetfile "Moteurs et alimentation.kicad_sch")
 		(attr through_hole)
@@
 			(layers "*.Cu" "*.Mask")
 			(remove_unused_layers no)
-			(net 13 "/Moteurs et alimentation/GND")
+			(net 14 "/Moteurs/GND")
 			(pinfunction "GND")
 			(pintype "power_in")
@@
 			(layers "*.Cu" "*.Mask")
 			(remove_unused_layers no)
-			(net 14 "Net-(LM1-IN-)")
+			(net 15 "Net-(J5-Pin_5)")
 			(pinfunction "GND")
 			(pintype "power_in")
@@
 			(layers "*.Cu" "*.Mask")
 			(remove_unused_layers no)
-			(net 15 "/Moteurs et alimentation/EN")
+			(net 20 "/Moteurs/EN")
 			(pinfunction "~{EN}")
 			(pintype "input")
@@
 			(layers "*.Cu" "*.Mask")
 			(remove_unused_layers no)
-			(net 6 "/Moteurs et alimentation/M0")
+			(net 6 "/Moteurs/M0")
 			(pinfunction "M0")
 			(pintype "input")
@@
 			(layers "*.Cu" "*.Mask")
 			(remove_unused_layers no)
-			(net 5 "/Moteurs et alimentation/M1")
+			(net 5 "/Moteurs/M1")
 			(pinfunction "M1")
 			(pintype "input")
@@
 			(layers "*.Cu" "*.Mask")
 			(remove_unused_layers no)
-			(net 11 "/Moteurs et alimentation/M2")
+			(net 11 "/Moteurs/M2")
 			(pinfunction "M2")
 			(pintype "input")
@@
 			(layers "*.Cu" "*.Mask")
 			(remove_unused_layers no)
-			(net 3 "/Moteurs et alimentation/RST{slash}SLP")
+			(net 3 "/Moteurs/RST{slash}SLP")
 			(pinfunction "~{RST}")
 			(pintype "input")
@@
 			(layers "*.Cu" "*.Mask")
 			(remove_unused_layers no)
-			(net 3 "/Moteurs et alimentation/RST{slash}SLP")
+			(net 3 "/Moteurs/RST{slash}SLP")
 			(pinfunction "~{SLP}")
 			(pintype "input")
@@
 			(layers "*.Cu" "*.Mask")
 			(remove_unused_layers no)
-			(net 12 "/Moteurs et alimentation/ALT{slash}STEP")
+			(net 12 "/Moteurs/ALT{slash}STEP")
 			(pinfunction "STEP")
 			(pintype "input")
@@
 			(layers "*.Cu" "*.Mask")
 			(remove_unused_layers no)
-			(net 8 "/Moteurs et alimentation/ALT{slash}DIR")
+			(net 8 "/Moteurs/ALT{slash}DIR")
 			(pinfunction "DIR")
 			(pintype "input")
