File: KiCad/Main/main.kicad_sch (KiCad schematic)
At the start: 16 parts, among them J1 Conn_01x02_Pin, J3 Vers Display, J8 RJ45, SW2 SW_DPST_x2, SW3 SW_DPST, SW4 SW_DPST_x2, U5 ESP32-S3-DevKitC

Commit message: ok
Parts:
- removed J1: Conn_01x02_Pin, symbol Connector:Conn_01x02_Pin
- removed J8: RJ45, Connector_RJ:RJ45_Amphenol_54602-x08_Horizontal, symbol Connector:RJ45
Connections:
- net RST: no longer U5.27 (GPIO21)
- net INT: no longer names the net of U5.19 (GPIO13/ADC2_CH2)
- net SCL: no longer names the net of U5.15 (GPIO9/ADC1_CH8)
- net SDA: no longer names the net of U5.12 (GPIO8/ADC1_CH7)
Other:
- sheet BNO085 renamed Capteurs
- sheet GMT020-02 renamed Display
